File: motor_i_enkoder.kicad_sch (KiCad schematic)
At the start: 13 parts, among them J7 Conn_02x06_Odd_Even, M1 JGB37-520, U4 L298N

Commit message: wszystko powinno dzialac. Trzeba zrobic podzial
Parts:
- added H10, H11, H12, H9: MountingHole, MountingHole:MountingHole_3.2mm_M3_DIN965_Pad_TopBottom, symbol Mechanical:MountingHole
- C11: footprint Capacitor_THT:CP_Axial_L10.0mm_D4.5mm_P15.00mm_Horizontal -> Capacitor_SMD:C_Elec_6.3x7.7; KiLib_Generator (none) -> capacitor/THT/other
- C12: footprint Capacitor_SMD:C_0805_2012Metric -> Capacitor_SMD:C_0805_2012Metric_Pad1.18x1.45mm_HandSolder; KiLib_Generator (none) -> SMD_2terminal_chip_molded
- D4, D5, D6, D7: footprint Diode_THT:D_DO-41_SOD81_P10.16mm_Horizontal -> Diode_SMD:D_SMA; KiLib_Generator (none) -> diode/THT
- J7: KiLib_Generator (none) -> connector/pin_header_socket
- L4: footprint Inductor_SMD:L_0805_2012Metric -> Inductor_SMD:L_Bourns_SRR1260; KiLib_Generator (none) -> SMD_2terminal_chip_molded
- M1: KiLib_Generator (none) -> terminal_block/Metz_Connect
- R10, R9: footprint Resistor_SMD:R_0805_2012Metric -> Resistor_SMD:R_1206_3216Metric_Pad1.30x1.75mm_HandSolder; KiLib_Generator (none) -> SMD_2terminal_chip_molded
- U4: KiLib_Generator (none) -> package/TO_SOT/THT
Connections:
- net 12V renamed 12V_2
- net CPU_GND renamed CPU_GND_2
- net DRIVER IN1 renamed DRIVER_IN1_1
- net DRIVER IN2 renamed DRIVER_IN2_1
- net DRIVER IN3 renamed unconnected-(J7-Pin_8-Pad8)
- net unconnected-(J7-Pin_8-Pad8): no longer U4.10 (IN3)
- net DRIVER IN4 renamed unconnected-(J7-Pin_10-Pad10)
- net unconnected-(J7-Pin_10-Pad10): no longer U4.12 (IN4)
- net ENC A renamed ENC_A_1
- net ENC B renamed ENC_B_1
- net GND renamed GND_2
- net PWM A renamed PWM_A_1
- net Vcc renamed Vcc_2
- net Vdd renamed Vdd_2
- new net unconnected-(U4-IN3-Pad10): U4.10 (IN3)
- new net unconnected-(U4-IN4-Pad12): U4.12 (IN4)
