File: sd_i_fram.kicad_sch (KiCad schematic)
At the start: 11 parts, among them J5 Conn_02x05_Odd_Even, J6 Goodram M1AA microSD 16GB 100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

Commit message: Niedziela
Parts:
- added H5, H6, H7, H8: MountingHole, MountingHole:MountingHole_3.2mm_M3_DIN965_Pad_TopBottom, symbol Mechanical:MountingHole
- C10, C9: footprint (none) -> Capacitor_SMD:C_0805_2012Metric_Pad1.18x1.45mm_HandSolder; KiLib_Generator (none) -> SMD_2terminal_chip_molded
- FRAM1: KiLib_Generator (none) -> package/gullwing
- J5: footprint (none) -> Connector_PinSocket_2.00mm:PinSocket_2x05_P2.00mm_Vertical_SMD; KiLib_Generator (none) -> connector/pin_header_socket
- J6: value Goodram M1AA microSD 16GB 100MB/s UHS-I klasa 10 z adapterem -> Molex 104031; footprint (none) -> Connector_Card:microSD_HC_Hirose_DM3D-SF
- R3, R4, R5, R6, R7, R8: footprint (none) -> Resistor_SMD:R_1206_3216Metric_Pad1.30x1.75mm_HandSolder; KiLib_Generator (none) -> SMD_2terminal_chip_molded
Connections:
- net #FRAM CS renamed ~{FRAM_CS_2}
- net #SD CS renamed ~{SD_CS_2}
- net GND_CPU renamed GND_CPU_1
- net MISO renamed MISO_2
- net MOSI renamed MOSI_2
- net SCK renamed SCK_2
- net VDD renamed VDD_1
Other:
- note added: "CZYTNIK MIKRO SD"
- note added: "FRAM"
- note removed: "VCC ma 5V VDD ma 3.3V lub 1.8V"
- moved on the sheet: C10, C9, FRAM1, J6, R3, R4, R5, R6, R7, R8
