File: sd_i_fram.kicad_sch (KiCad schematic)
At the start: 11 parts, among them J5 Conn_02x05_Odd_Even, J6 Molex 104031

Commit message: wszystko powinno dzialac. Trzeba zrobic podzial
Parts:
- added H5, H6, H7, H8: MountingHole, MountingHole:MountingHole_3.2mm_M3_DIN965_Pad_TopBottom, symbol Mechanical:MountingHole
- C10, C9: footprint Capacitor_SMD:C_0805_2012Metric -> Capacitor_SMD:C_0805_2012Metric_Pad1.18x1.45mm_HandSolder; KiLib_Generator (none) -> SMD_2terminal_chip_molded
- FRAM1: KiLib_Generator (none) -> package/gullwing
- J5: footprint Connector_PinHeader_2.54mm:PinHeader_2x06_P2.54mm_Vertical -> Connector_PinHeader_2.54mm:PinHeader_2x05_P2.54mm_Vertical_SMD; KiLib_Generator (none) -> connector/pin_header_socket
- R3, R4, R5, R6, R7, R8: footprint Resistor_SMD:R_0805_2012Metric -> Resistor_SMD:R_1206_3216Metric_Pad1.30x1.75mm_HandSolder; KiLib_Generator (none) -> SMD_2terminal_chip_molded
Connections:
- net GND_CPU renamed GND_CPU_1
- net MISO renamed MISO_2
- net MOSI renamed MOSI_2
- net SCK renamed SCK_2
- net VDD renamed VDD_1
- net /FRAM CS renamed ~{FRAM_CS_2}
- net /SD CS renamed ~{SD_CS_2}
