File: smiw_proj.kicad_pcb (KiCad board)
At the start: 2 copper layers, 104.4 x 97.8 mm, 60 parts, among them J1 Conn_02x06_Odd_Even, J2 Conn_02x05_Odd_Even, J3 Conn_01x02, J4 Conn_01x02, J5 Conn_02x05_Odd_Even, J6 Molex 104031, J7 Conn_02x06_Odd_Even, M1 JGB37-520, SW1 SW_Push, U1 LM2596S-5, U2 M5 Stamp-S3, U3 LD1117S33TR_SOT223, U4 L298N

Commit message: rezystor
Parts:
- removed H10, H11, H12, H5, H6, H7, H8, H9: MountingHole, MountingHole:MountingHole_3.2mm_M3_DIN965_Pad_TopBottom
- added R11: 0, Resistor_SMD:R_0805_2012Metric, F.Cu at (20.0, 50.4)
- C10, C12, C9: footprint Capacitor_SMD:C_0805_2012Metric_Pad1.18x1.45mm_HandSolder -> Capacitor_SMD:C_0805_2012Metric
- C11: footprint Capacitor_SMD:C_Elec_6.3x7.7 -> Capacitor_THT:CP_Axial_L10.0mm_D4.5mm_P15.00mm_Horizontal
- D4, D5, D6, D7: footprint Diode_SMD:D_SMA -> Diode_THT:D_DO-41_SOD81_P10.16mm_Horizontal
- J2: footprint Connector_PinSocket_1.00mm:PinSocket_2x05_P1.00mm_Vertical_SMD -> Connector_PinSocket_2.54mm:PinSocket_2x05_P2.54mm_Vertical_SMD
- J5: footprint Connector_PinSocket_2.00mm:PinSocket_2x05_P2.00mm_Vertical_SMD -> Connector_PinHeader_2.54mm:PinHeader_2x06_P2.54mm_Vertical
- L4: footprint Inductor_SMD:L_Bourns_SRR1260 -> Inductor_SMD:L_0805_2012Metric
- R10, R3, R4, R5, R6, R7, R8, R9: footprint Resistor_SMD:R_1206_3216Metric_Pad1.30x1.75mm_HandSolder -> Resistor_SMD:R_0805_2012Metric
- moved U2 14.8 mm to (43.0, 32.6)
- moved J2 14.0 mm to (71.2, 51.4), turned to -90 degrees
- moved C2 0.93 mm to (64.1, 22.6)
Connections:
- net /~{FRAM_CS_2} renamed //FRAM CS
- net /~{SD_CS_2} renamed //SD CS
- net VDD_2 renamed VDD
- C10 pad 2: GND_CPU_2 -> GND_CPU
- C11 pad 2: GND_1 -> GND
- C12 pad 2: GND_1 -> GND
- C7 pad 2: GND -> GND_CPU
- C8 pad 1: GND -> GND_CPU
- C9 pad 1: GND_CPU_2 -> GND_CPU
- D6 pad 2: GND_1 -> GND
- D7 pad 2: GND_1 -> GND
- FRAM1 pad 2: /MISO_2 -> /MISO
- FRAM1 pad 4: GND_CPU_2 -> GND_CPU
- FRAM1 pad 5: /MOSI_2 -> /MOSI
- FRAM1 pad 6: /SCK_2 -> /SCK
- J2 pad 3: GND -> GND_CPU
- J2 pad 5: GND -> GND_CPU
- J2 pad 7: GND -> GND_CPU
- J2 pad 9: GND -> GND_CPU
- J5 pad 2: /MOSI_2 -> /MOSI
- J5 pad 3: GND_CPU_2 -> GND_CPU
- J5 pad 4: /MISO_2 -> /MISO
- J5 pad 5: GND_CPU_2 -> GND_CPU
- J5 pad 6: /SCK_2 -> /SCK
- J5 pad 7: GND_CPU_2 -> GND_CPU
- J5 pad 9: GND_CPU_2 -> GND_CPU
- J6 pad 3: /MOSI_2 -> /MOSI
- J6 pad 5: /SCK_2 -> /SCK
- J6 pad 6: GND_CPU_2 -> GND_CPU
- J6 pad 7: /MISO_2 -> /MISO
- J6 pad SH: GND_CPU_2 -> GND_CPU
- J7 pad 1: 12V_1 -> 12V
- J7 pad 10: unconnected-(J7-Pin_10-Pad10) -> /DRIVER IN4
- J7 pad 11: /ENC_A_1 -> /ENC A
- J7 pad 12: /ENC_B_1 -> /ENC B
- J7 pad 2: /DRIVER_IN1_1 -> /DRIVER IN1
- J7 pad 3: Vcc_1 -> Vcc
- J7 pad 4: /DRIVER_IN2_1 -> /DRIVER IN2
- J7 pad 5: Vdd_1 -> Vdd
- J7 pad 6: /PWM_A_1 -> /PWM A
- J7 pad 7: GND_1 -> GND
- J7 pad 8: unconnected-(J7-Pin_8-Pad8) -> /DRIVER IN3
- J7 pad 9: CPU_GND_1 -> CPU_GND
- L4 pad 1: 12V_1 -> 12V
- R10 pad 1: /ENC_A_1 -> /ENC A
- R10 pad 2: Vdd_1 -> Vdd
- R7 pad 2: /MOSI_2 -> /MOSI
- R8 pad 2: /MISO_2 -> /MISO
- R9 pad 1: /ENC_B_1 -> /ENC B
- R9 pad 2: Vdd_1 -> Vdd
- RotatoryEncoder1 pad A: /ENC_A_1 -> /ENC A
- RotatoryEncoder1 pad B: /ENC_B_1 -> /ENC B
- RotatoryEncoder1 pad C: CPU_GND_1 -> CPU_GND
- SW1 pad 2: GND -> GND_CPU
- U2 pad 11: GND -> GND_CPU
- U2 pad 18: GND -> GND_CPU
- U4 pad 1: GND_1 -> GND
- U4 pad 10: unconnected-(U4-IN3-Pad10) -> /DRIVER IN3
- U4 pad 11: GND_1 -> GND
- U4 pad 12: unconnected-(U4-IN4-Pad12) -> /DRIVER IN4
- U4 pad 15: GND_1 -> GND
- U4 pad 4: Vcc_1 -> Vcc
- U4 pad 5: /DRIVER_IN1_1 -> /DRIVER IN1
- U4 pad 6: /PWM_A_1 -> /PWM A
- U4 pad 7: /DRIVER_IN2_1 -> /DRIVER IN2
- U4 pad 8: GND_1 -> GND
Routing:
- net (no net): track 0.00 -> 94.3 mm, vias 0 -> 2
- net /MISO: track 30.8 -> 94.7 mm, vias 0 -> 4
- net /ENC_A_1: track 63.5 -> 0.00 mm, vias 6 -> 0
- net 12V: track 33.0 -> 92.2 mm, vias 0 -> 4
- net /MOSI: track 33.2 -> 91.0 mm, vias 2 -> 9
- net 12V_1: track 54.6 -> 0.00 mm, vias 3 -> 0
- net /DRIVER_IN2_1: track 54.2 -> 0.00 mm
- net GND: track 0.00 -> 48.6 mm, vias 0 -> 5
- net /MISO_2: track 48.5 -> 0.00 mm, vias 2 -> 0
- net /ENC_B_1: track 46.4 -> 0.00 mm, vias 3 -> 0
- net /MOSI_2: track 42.4 -> 0.00 mm, vias 5 -> 0
- net /SCK: track 27.6 -> 69.5 mm, vias 2 -> 6
- net CPU_GND: track 0.00 -> 35.3 mm
- net Vdd_1: track 34.7 -> 0.00 mm, vias 1 -> 0
- net /PWM_A_1: track 30.9 -> 0.00 mm
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- added copper zone on B.Cu, net (none)
- added copper zone on F.Cu, net (none)
- removed copper zone on B.Cu, net CPU_GND_1
- removed copper zone on F.Cu, net GND_1
- removed copper zone on F.Cu, net GND_CPU_2

Commit message: Niedziela
Parts:
- added H10: MountingHole, MountingHole:MountingHole_3.2mm_M3_DIN965_Pad_TopBottom, F.Cu at (115.6, 73.7)
- added H11: MountingHole, MountingHole:MountingHole_3.2mm_M3_DIN965_Pad_TopBottom, F.Cu at (64.8, 106.7)
- added H12: MountingHole, MountingHole:MountingHole_3.2mm_M3_DIN965_Pad_TopBottom, F.Cu at (115.6, 106.7)
- added H5: MountingHole, MountingHole:MountingHole_3.2mm_M3_DIN965_Pad_TopBottom, F.Cu at (19.1, 73.7)
- added H6: MountingHole, MountingHole:MountingHole_3.2mm_M3_DIN965_Pad_TopBottom, F.Cu at (50.8, 73.7)
- added H7: MountingHole, MountingHole:MountingHole_3.2mm_M3_DIN965_Pad_TopBottom, F.Cu at (19.1, 106.7)
- added H8: MountingHole, MountingHole:MountingHole_3.2mm_M3_DIN965_Pad_TopBottom, F.Cu at (50.8, 106.7)
- added H9: MountingHole, MountingHole:MountingHole_3.2mm_M3_DIN965_Pad_TopBottom, F.Cu at (64.8, 73.7)
- C10, C12, C9: footprint Capacitor_SMD:C_0805_2012Metric -> Capacitor_SMD:C_0805_2012Metric_Pad1.18x1.45mm_HandSolder
- C11: footprint Capacitor_THT:CP_Axial_L10.0mm_D4.5mm_P15.00mm_Horizontal -> Capacitor_SMD:C_Elec_6.3x7.7
- D4, D5, D6, D7: footprint Diode_THT:D_DO-41_SOD81_P10.16mm_Horizontal -> Diode_SMD:D_SMA
- J5: footprint Connector_PinHeader_2.54mm:PinHeader_2x06_P2.54mm_Vertical -> Connector_PinSocket_2.00mm:PinSocket_2x05_P2.00mm_Vertical_SMD
- L4: footprint Inductor_SMD:L_0805_2012Metric -> Inductor_SMD:L_Bourns_SRR1260
- R10, R11, R3, R4, R5, R6, R7, R8, R9: footprint Resistor_SMD:R_0805_2012Metric -> Resistor_SMD:R_1206_3216Metric_Pad1.30x1.75mm_HandSolder
- U2: footprint Library2:Stamp-S3_PIN1.27_Socket -> Library:M5Stamp-S3
- moved R11 1.72 mm to (21.6, 51.1)
Connections:
- net //FRAM CS renamed /~{FRAM_CS_2}
- net //SD CS renamed /~{SD_CS_2}
- net VDD renamed VDD_1
- C10 pad 2: GND_CPU -> GND_CPU_1
- C11 pad 2: GND -> GND_2
- C12 pad 2: GND -> GND_2
- C9 pad 1: GND_CPU -> GND_CPU_1
- D6 pad 2: GND -> GND_2
- D7 pad 2: GND -> GND_2
- FRAM1 pad 2: /MISO -> /MISO_2
- FRAM1 pad 4: GND_CPU -> GND_CPU_1
- FRAM1 pad 5: /MOSI -> /MOSI_2
- FRAM1 pad 6: /SCK -> /SCK_2
- J1 pad 9: CPU_GND -> GND_CPU
- J5 pad 2: /MOSI -> /MOSI_2
- J5 pad 3: GND_CPU -> GND_CPU_1
- J5 pad 4: /MISO -> /MISO_2
- J5 pad 5: GND_CPU -> GND_CPU_1
- J5 pad 6: /SCK -> /SCK_2
- J5 pad 7: GND_CPU -> GND_CPU_1
- J5 pad 9: GND_CPU -> GND_CPU_1
- J6 pad 3: /MOSI -> /MOSI_2
- J6 pad 5: /SCK -> /SCK_2
- J6 pad 6: GND_CPU -> GND_CPU_1
- J6 pad 7: /MISO -> /MISO_2
- J6 pad SH: GND_CPU -> GND_CPU_1
- J7 pad 1: 12V -> 12V_2
- J7 pad 10: /DRIVER IN4 -> /unconnected-(J7-Pin_10-Pad10)
- J7 pad 11: /ENC A -> /ENC_A_1
- J7 pad 12: /ENC B -> /ENC_B_1
- J7 pad 2: /DRIVER IN1 -> /DRIVER_IN1_1
- J7 pad 3: Vcc -> Vcc_2
- J7 pad 4: /DRIVER IN2 -> /DRIVER_IN2_1
- J7 pad 5: Vdd -> Vdd_2
- J7 pad 6: /PWM A -> /PWM_A_1
- J7 pad 7: GND -> GND_2
- J7 pad 8: /DRIVER IN3 -> /unconnected-(J7-Pin_8-Pad8)
- J7 pad 9: CPU_GND -> CPU_GND_2
- L4 pad 1: 12V -> 12V_2
- R10 pad 1: /ENC A -> /ENC_A_1
- R10 pad 2: Vdd -> Vdd_2
- R11 pad 1: CPU_GND -> GND_CPU
- R7 pad 2: /MOSI -> /MOSI_2
- R8 pad 2: /MISO -> /MISO_2
- R9 pad 1: /ENC B -> /ENC_B_1
- R9 pad 2: Vdd -> Vdd_2
- RotatoryEncoder1 pad A: /ENC A -> /ENC_A_1
- RotatoryEncoder1 pad B: /ENC B -> /ENC_B_1
- RotatoryEncoder1 pad C: CPU_GND -> CPU_GND_2
- U4 pad 1: GND -> GND_2
- U4 pad 10: /DRIVER IN3 -> /unconnected-(U4-IN3-Pad10)
- U4 pad 11: GND -> GND_2
- U4 pad 12: /DRIVER IN4 -> /unconnected-(U4-IN4-Pad12)
- U4 pad 15: GND -> GND_2
- U4 pad 4: Vcc -> Vcc_2
- U4 pad 5: /DRIVER IN1 -> /DRIVER_IN1_1
- U4 pad 6: /PWM A -> /PWM_A_1
- U4 pad 7: /DRIVER IN2 -> /DRIVER_IN2_1
- U4 pad 8: GND -> GND_2
Routing:
- net (no net): track 94.3 -> 0.00 mm, vias 2 -> 0
- net 12V_2: track 0.00 -> 56.0 mm, vias 0 -> 3
- net 12V: track 92.2 -> 36.2 mm, vias 4 -> 1
- net /MISO: track 94.7 -> 46.2 mm, vias 4 -> 2
- net /MISO_2: track 0.00 -> 48.5 mm, vias 0 -> 2
- net /ENC_B_1: track 0.00 -> 46.2 mm, vias 0 -> 2
- net /ENC B: track 60.0 -> 13.8 mm, vias 3 -> 1
- net /MOSI_2: track 0.00 -> 42.4 mm, vias 0 -> 5
- net /MOSI: track 91.0 -> 48.7 mm, vias 9 -> 4
- net GND: track 48.6 -> 6.96 mm, vias 5 -> 0
- net /ENC_A_1: track 0.00 -> 40.3 mm, vias 0 -> 1
- net CPU_GND: track 35.3 -> 0.00 mm
- net /PWM A: track 37.4 -> 6.33 mm
- net /PWM_A_1: track 0.00 -> 30.9 mm, vias 0 -> 2
- net /SCK: track 69.5 -> 39.8 mm, vias 6 -> 2
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- added copper zone on B.Cu, net CPU_GND_2
- added copper zone on F.Cu, net GND_2
- added copper zone on B.Cu, net GND_CPU
- added copper zone on F.Cu, net GND_CPU_1
- removed copper zone on B.Cu, net (none)
- removed copper zone on F.Cu, net (none)
Other:
- outline, holes or cut-outs redrawn
