File: smiw_proj.kicad_pcb (KiCad board)
At the start: 2 copper layers, 115.6 x 104.1 mm, 60 parts, among them J1 Conn_02x06_Odd_Even, J2 Conn_02x05_Odd_Even, J3 Conn_01x02, J4 Conn_01x02, J5 Conn_02x05_Odd_Even, J6 Molex 104031, J7 Conn_02x06_Odd_Even, M1 JGB37-520, SW1 SW_Push, U1 LM2596S-5, U2 M5 Stamp-S3, U3 LD1117S33TR_SOT223, U4 L298N

Commit message: pcb dobrze zdaniem michala (to nie ma sensu)
Parts:
- removed REF** (x12): MountingHole_2.1mm, MountingHole:MountingHole_2.1mm
- added H1: MountingHole, MountingHole:MountingHole_3.2mm_M3_DIN965_Pad_TopBottom, F.Cu at (19.6, 17.0)
- added H10: MountingHole, MountingHole:MountingHole_3.2mm_M3_DIN965_Pad_TopBottom, F.Cu at (64.5, 106.7)
- added H11: MountingHole, MountingHole:MountingHole_3.2mm_M3_DIN965_Pad_TopBottom, F.Cu at (115.3, 73.7)
- added H12: MountingHole, MountingHole:MountingHole_3.2mm_M3_DIN965_Pad_TopBottom, F.Cu at (115.3, 106.7)
- added H2: MountingHole, MountingHole:MountingHole_3.2mm_M3_DIN965_Pad_TopBottom, F.Cu at (115.6, 16.5)
- added H3: MountingHole, MountingHole:MountingHole_3.2mm_M3_DIN965_Pad_TopBottom, F.Cu at (19.1, 58.4)
- added H4: MountingHole, MountingHole:MountingHole_3.2mm_M3_DIN965_Pad_TopBottom, F.Cu at (115.6, 58.4)
- added H5: MountingHole, MountingHole:MountingHole_3.2mm_M3_DIN965_Pad_TopBottom, F.Cu at (18.8, 73.7)
- added H6: MountingHole, MountingHole:MountingHole_3.2mm_M3_DIN965_Pad_TopBottom, F.Cu at (18.8, 106.7)
- added H7: MountingHole, MountingHole:MountingHole_3.2mm_M3_DIN965_Pad_TopBottom, F.Cu at (50.5, 73.7)
- added H8: MountingHole, MountingHole:MountingHole_3.2mm_M3_DIN965_Pad_TopBottom, F.Cu at (50.5, 106.7)
- added H9: MountingHole, MountingHole:MountingHole_3.2mm_M3_DIN965_Pad_TopBottom, F.Cu at (64.5, 73.7)
- J1: footprint Connector_PinSocket_1.00mm:PinSocket_2x05_P1.00mm_Vertical_SMD -> Connector_PinHeader_2.54mm:PinHeader_2x06_P2.54mm_Vertical
- J2: footprint Connector_PinSocket_1.00mm:PinSocket_2x05_P1.00mm_Vertical_SMD -> Connector_PinSocket_2.54mm:PinSocket_2x05_P2.54mm_Vertical_SMD
- J5: footprint Connector_PinHeader_2.54mm:PinHeader_2x06_P2.54mm_Vertical -> Connector_PinSocket_2.00mm:PinSocket_2x05_P2.00mm_Vertical_SMD
- U2: footprint Library2:Stamp-S3_PIN1.27_Socket -> Library:M5Stamp-S3
- moved J1 82.2 mm to (27.0, 45.7)
- moved C10 70.1 mm to (39.1, 97.8), turned to 0 degrees
- moved C9 49.0 mm to (21.5, 83.8)
- moved J2 48.1 mm to (71.2, 51.4), turned to -90 degrees
- moved C11 34.4 mm to (89.9, 77.5)
- moved R9 29.3 mm to (79.7, 96.2)
- moved R10 28.1 mm to (83.5, 96.2)
- moved RotatoryEncoder1 23.6 mm to (96.2, 77.5)
- moved L4 19.1 mm to (102.8, 95.3)
- moved J7 17.4 mm to (70.8, 78.8)
- moved C12 16.3 mm to (75.9, 94.0)
- moved L3 15.2 mm to (110.8, 29.4), turned to -90 degrees
- moved U2 15.0 mm to (43.0, 32.6)
- moved U4 13.9 mm to (74.6, 91.5)
- moved J5 12.3 mm to (30.0, 75.5)
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Connections:
- net //FRAM CS renamed /~{FRAM_CS_2}
- net //SD CS renamed /~{SD_CS_2}
- net VDD renamed VDD_2
- C10 pad 2: GND -> GND_CPU_2
- C11 pad 2: GND -> GND_1
- C12 pad 2: GND -> GND_1
- C9 pad 1: GND -> GND_CPU_2
- D6 pad 2: GND -> GND_1
- D7 pad 2: GND -> GND_1
- FRAM1 pad 2: /MISO -> /MISO_2
- FRAM1 pad 4: GND -> GND_CPU_2
- FRAM1 pad 5: /MOSI -> /MOSI_2
- FRAM1 pad 6: /SCK -> /SCK_2
- J5 pad 2: /MOSI -> /MOSI_2
- J5 pad 3: GND -> GND_CPU_2
- J5 pad 4: /MISO -> /MISO_2
- J5 pad 5: GND -> GND_CPU_2
- J5 pad 6: /SCK -> /SCK_2
- J5 pad 7: GND -> GND_CPU_2
- J5 pad 9: GND -> GND_CPU_2
- J6 pad 3: /MOSI -> /MOSI_2
- J6 pad 5: /SCK -> /SCK_2
- J6 pad 6: GND -> GND_CPU_2
- J6 pad 7: /MISO -> /MISO_2
- J6 pad SH: GND -> GND_CPU_2
- J7 pad 1: 12V -> 12V_1
- J7 pad 10: /DRIVER IN4 -> unconnected-(J7-Pin_10-Pad10)
- J7 pad 11: /ENC A -> /ENC_A_1
- J7 pad 12: /ENC B -> /ENC_B_1
- J7 pad 2: /DRIVER IN1 -> /DRIVER_IN1_1
- J7 pad 3: Vcc -> Vcc_1
- J7 pad 4: /DRIVER IN2 -> /DRIVER_IN2_1
- J7 pad 5: Vdd -> Vdd_1
- J7 pad 6: /PWM A -> /PWM_A_1
- J7 pad 7: GND -> GND_1
- J7 pad 8: /DRIVER IN3 -> unconnected-(J7-Pin_8-Pad8)
- J7 pad 9: CPU_GND -> CPU_GND_1
- L4 pad 1: 12V -> 12V_1
- R10 pad 1: /ENC A -> /ENC_A_1
- R10 pad 2: Vdd -> Vdd_1
- R7 pad 2: /MOSI -> /MOSI_2
- R8 pad 2: /MISO -> /MISO_2
- R9 pad 1: /ENC B -> /ENC_B_1
- R9 pad 2: Vdd -> Vdd_1
- RotatoryEncoder1 pad A: /ENC A -> /ENC_A_1
- RotatoryEncoder1 pad B: /ENC B -> /ENC_B_1
- RotatoryEncoder1 pad C: CPU_GND -> CPU_GND_1
- U4 pad 1: GND -> GND_1
- U4 pad 10: /DRIVER IN3 -> unconnected-(U4-IN3-Pad10)
- U4 pad 11: GND -> GND_1
- U4 pad 12: /DRIVER IN4 -> unconnected-(U4-IN4-Pad12)
- U4 pad 15: GND -> GND_1
- U4 pad 4: Vcc -> Vcc_1
- U4 pad 5: /DRIVER IN1 -> /DRIVER_IN1_1
- U4 pad 6: /PWM A -> /PWM_A_1
- U4 pad 7: /DRIVER IN2 -> /DRIVER_IN2_1
- U4 pad 8: GND -> GND_1
Routing:
- net GND: track 214.7 -> 28.3 mm, vias 7 -> 3
- net /PWM A: track 136.7 -> 6.33 mm, vias 0 -> 2
- net Vcc: track 70.5 -> 180.2 mm, vias 1 -> 4
- net /DRIVER IN3: track 122.2 -> 18.8 mm
- net /DRIVER IN1: track 111.0 -> 11.6 mm, vias 3 -> 0
- net /~{FRAM CS}: track 114.7 -> 34.6 mm, vias 0 -> 4
- net Net-(D4-K): track 30.6 -> 107.6 mm, vias 0 -> 6
- net (no net): track 70.0 -> 0.00 mm, vias 7 -> 0
- net 12V_1: track 0.00 -> 56.0 mm, vias 0 -> 3
- net /MISO_2: track 0.00 -> 48.5 mm, vias 0 -> 2
- net /ENC_B_1: track 0.00 -> 46.2 mm, vias 0 -> 2
- net /~{SD CS}: track 0.00 -> 43.7 mm, vias 0 -> 5
- net VDD_2: track 121.1 -> 77.9 mm, vias 1 -> 0
- net Vdd: track 75.1 -> 117.8 mm, vias 1 -> 2
- net /MOSI_2: track 0.00 -> 42.4 mm, vias 0 -> 5
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- added copper zone on B.Cu, net CPU_GND_1
- added copper zone on F.Cu, net GND_1
- added copper zone on F.Cu, net GND_CPU_2
- removed copper zone on B.Cu, net GND
Other:
- board size 115.6 x 104.1 mm -> 104.4 x 97.8 mm

Commit message: s
Routing:
- net /ENC A: track 47.6 -> 21.3 mm
- added copper zone on B.Cu, net (none)
- removed copper zone on B.Cu, net CPU_GND_1
Changed lines of the file:
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@@
 		(sheetname "/")
 		(sheetfile "smiw_proj.kicad_sch")
+		(units
+			(unit
+				(name "A")
+				(pins "1" "2" "3" "4" "5" "6" "7" "8" "9" "10" "11" "12" "13" "14" "15"
+					"16" "17" "28" "27" "26" "25" "24" "23" "22" "21" "20" "19" "18"
+				)
+			)
+		)
 		(attr smd)
 		(duplicate_pad_numbers_are_jumpers no)
@@
 		(sheetname "/")
 		(sheetfile "smiw_proj.kicad_sch")
+		(units
+			(unit
+				(name "A")
+				(pins "1" "3" "5" "7" "9" "2" "4" "6" "8" "10")
+			)
+		)
 		(attr smd)
 		(duplicate_pad_numbers_are_jumpers no)
@@
 	)
 	(segment
-		(start 37.7 45.948529)
-		(end 37.348529 46.3)
-		(width 0.2)
-		(layer "F.Cu")
-		(net "/ENC A")
-	)
-	(segment
-		(start 34.413544 46.105082)
-		(end 34.154283 45.845821)
-		(width 0.2)
-		(layer "F.Cu")
-		(net "/ENC A")
-	)
-	(segment
-		(start 32.448003 47.35)
-		(end 33.193874 48.095871)
-		(width 0.2)
-		(layer "F.Cu")
-		(net "/ENC A")
-	)
-	(segment
-		(start 35.444233 45.955871)
-		(end 35.250738 46.149366)
-		(width 0.2)
-		(layer "F.Cu")
-		(net "/ENC A")
-	)
-	(segment
-		(start 35.62 44.905)
-		(end 35.336367 44.905)
-		(width 0.2)
-		(layer "F.Cu")
-		(net "/ENC A")
-	)
-	(segment
-		(start 34.283633 44.905)
-		(end 32.67032 44.905)
-		(width 0.2)
-		(layer "F.Cu")
-		(net "/ENC A")
-	)
-	(segment
-		(start 35.141371 47.639998)
-		(end 34.478629 47.639998)
-		(width 0.2)
-		(layer "F.Cu")
-		(net "/ENC A")
-	)
-	(segment
-		(start 36.851471 45.1)
-		(end 37.348529 45.1)
-		(width 0.2)
-		(layer "F.Cu")
-		(net "/ENC A")
-	)
-	(segment
-		(start 35.336367 44.905)
-		(end 35.264864 44.976503)
-		(width 0.2)
-		(layer "F.Cu")
-		(net "/ENC A")
-	)
-	(segment
-		(start 38.159999 44.815)
-		(end 35.71 44.815)
-		(width 0.2)
-		(layer "F.Cu")
-		(net "/ENC A")
-	)
-	(segment
-		(start 37.348529 45.1)
-		(end 37.7 45.451471)
-		(width 0.2)
-		(layer "F.Cu")
-		(net "/ENC A")
-	)
-	(segment
-		(start 34.478629 47.639998)
-		(end 34.01 47.171369)
-		(width 0.2)
-		(layer "F.Cu")
-		(net "/ENC A")
-	)
-	(segment
-		(start 39.668003 54.826997)
-		(end 39.668003 46.323003)
-		(width 0.2)
-		(layer "F.Cu")
-		(net "/ENC A")
-	)
-	(segment
-		(start 37.7 45.451471)
-		(end 37.7 45.948529)
-		(width 0.2)
-		(layer "F.Cu")
-		(net "/ENC A")
-	)
-	(segment
-		(start 34.01 46.508627)
-		(end 34.413544 46.105082)
-		(width 0.2)
-		(layer "F.Cu")
-		(net "/ENC A")
-	)
-	(segment
-		(start 32.448003 45.127317)
-		(end 32.448003 47.35)
-		(width 0.2)
-		(layer "F.Cu")
-		(net "/ENC A")
-	)
-	(segment
-		(start 37.348529 46.3)
-		(end 36.851471 46.3)
-		(width 0.2)
-		(layer "F.Cu")
-		(net "/ENC A")
-	)
-	(segment
-		(start 39.668003 46.323003)
-		(end 38.159999 44.815)
-		(width 0.2)
-		(layer "F.Cu")
-		(net "/ENC A")
-	)
-	(segment
-		(start 34.154283 45.845821)
-		(end 34.154283 45.265921)
-		(width 0.2)
-		(layer "F.Cu")
-		(net "/ENC A")
-	)
-	(segment
-		(start 34.695 59.8)
-		(end 39.668003 54.826997)
-		(width 0.2)
-		(layer "F.Cu")
-		(net "/ENC A")
-	)
-	(segment
-		(start 34.399418 45.020785)
-		(end 34.283633 44.905)
-		(width 0.2)
-		(layer "F.Cu")
-		(net "/ENC A")
-	)
-	(segment
 		(start 26.968003 58.42)
 		(end 28.348003 59.8)
@@
 	)
 	(segment
-		(start 35.444233 45.155871)
-		(end 36.7956 45.155871)
-		(width 0.2)
-		(layer "F.Cu")
-		(net "/ENC A")
-	)
-	(segment
-		(start 35.264864 44.976503)
-		(end 35.444233 45.155871)
-		(width 0.2)
-		(layer "F.Cu")
-		(net "/ENC A")
-	)
-	(segment
-		(start 35.71 44.815)
-		(end 35.62 44.905)
-		(width 0.2)
-		(layer "F.Cu")
-		(net "/ENC A")
-	)
-	(segment
-		(start 34.01 47.171369)
-		(end 34.01 46.508627)
-		(width 0.2)
-		(layer "F.Cu")
-		(net "/ENC A")
-	)
-	(segment
-		(start 33.193874 48.095871)
+		(start 36.35 49.591588)
 		(end 34.854283 48.095871)
 		(width 0.2)
@@
 	)
 	(segment
-		(start 36.507342 45.955871)
-		(end 35.444233 45.955871)
-		(width 0.2)
-		(layer "F.Cu")
-		(net "/ENC A")
-	)
-	(segment
-		(start 32.67032 44.905)
-		(end 32.448003 45.127317)
-		(width 0.2)
-		(layer "F.Cu")
-		(net "/ENC A")
-	)
-	(segment
-		(start 34.154283 45.265921)
-		(end 34.399418 45.020785)
-		(width 0.2)
-		(layer "F.Cu")
-		(net "/ENC A")
-	)
-	(segment
-		(start 35.61 46.508627)
-		(end 35.61 47.171369)
-		(width 0.2)
-		(layer "F.Cu")
-		(net "/ENC A")
-	)
-	(segment
-		(start 36.851471 46.3)
-		(end 36.507342 45.955871)
-		(width 0.2)
-		(layer "F.Cu")
-		(net "/ENC A")
-	)
-	(segment
 		(start 28.348003 59.8)
 		(end 34.695 59.8)
@@
 	)
 	(segment
-		(start 36.7956 45.155871)
-		(end 36.851471 45.1)
-		(width 0.2)
-		(layer "F.Cu")
-		(net "/ENC A")
-	)
-	(segment
-		(start 35.61 47.171369)
-		(end 35.141371 47.639998)
+		(start 34.695 59.8)
+		(end 36.35 58.145)
 		(width 0.2)
 		(layer "F.Cu")
@@
 	)
 	(segment
-		(start 35.250738 46.149366)
-		(end 35.61 46.508627)
+		(start 36.35 58.145)
+		(end 36.35 49.591588)
 		(width 0.2)
 		(layer "F.Cu")
@@
 	)
 	(zone
-		(net "CPU_GND_1")
 		(layer "B.Cu")
 		(name "cpu_gnd")

Commit message: wszystko powinno dzialac. Trzeba zrobic podzial
Parts:
- added R11: 0, Resistor_SMD:R_1206_3216Metric_Pad1.30x1.75mm_HandSolder, F.Cu at (21.6, 51.1)
- J1: footprint Connector_PinHeader_2.54mm:PinHeader_2x06_P2.54mm_Vertical -> Connector_PinSocket_2.54mm:PinSocket_2x06_P2.54mm_Vertical
- J5: footprint Connector_PinSocket_2.00mm:PinSocket_2x05_P2.00mm_Vertical_SMD -> Connector_PinHeader_2.54mm:PinHeader_2x05_P2.54mm_Vertical_SMD
- moved H11 61.7 mm to (65.8, 110.6)
- moved H10 59.7 mm to (116.6, 77.6)
- moved H7 51.4 mm to (17.3, 112.9)
- moved H6 42.4 mm to (49.1, 77.2)
- moved J1 12.5 mm to (27.1, 58.2), turned to 180 degrees
- moved C10 6.48 mm to (37.4, 104.0)
- moved FRAM1 6.48 mm to (25.3, 91.7)
- moved J6 6.48 mm to (28.0, 105.4)
- moved R3 6.48 mm to (42.5, 89.1)
- moved R4 6.48 mm to (42.5, 86.1)
- moved R5 6.48 mm to (42.5, 83.2)
- moved R6 6.48 mm to (42.4, 97.3)
- moved R7 6.48 mm to (42.4, 94.4)
- moved R8 6.48 mm to (42.4, 91.4)
- moved C9 6.48 mm to (19.8, 90.1)
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Connections:
- net 12V_1 renamed 12V_2
- net CPU_GND_1 renamed CPU_GND_2
- net GND_1 renamed GND_2
- net GND_CPU_2 renamed GND_CPU_1
- net VDD_2 renamed VDD_1
- net Vcc_1 renamed Vcc_2
- net Vdd_1 renamed Vdd_2
- C7 pad 2: GND -> GND_CPU
- C8 pad 1: GND -> GND_CPU
- J1 pad 9: CPU_GND -> GND_CPU
- J2 pad 3: GND -> GND_CPU
- J2 pad 5: GND -> GND_CPU
- J2 pad 7: GND -> GND_CPU
- J2 pad 9: GND -> GND_CPU
- J7 pad 10: unconnected-(J7-Pin_10-Pad10) -> /unconnected-(J7-Pin_10-Pad10)
- J7 pad 8: unconnected-(J7-Pin_8-Pad8) -> /unconnected-(J7-Pin_8-Pad8)
- SW1 pad 2: GND -> GND_CPU
- U2 pad 11: GND -> GND_CPU
- U2 pad 18: GND -> GND_CPU
- U4 pad 10: unconnected-(U4-IN3-Pad10) -> /unconnected-(U4-IN3-Pad10)
- U4 pad 12: unconnected-(U4-IN4-Pad12) -> /unconnected-(U4-IN4-Pad12)
Routing:
- net GND: track 28.3 -> 6.42 mm, vias 3 -> 0
- net 12V: track 36.2 -> 54.6 mm
- net /DRIVER IN1: track 11.6 -> 24.2 mm, vias 0 -> 3
- net /ENC A: track 21.3 -> 10.9 mm
- net /DRIVER IN2: track 13.3 -> 20.9 mm, vias 0 -> 1
- net Vcc: track 180.2 -> 172.7 mm, vias 4 -> 3
- net /~{FRAM_CS_2}: track 24.5 -> 31.5 mm, vias 2 -> 3
- net /DRIVER IN4: track 12.0 -> 5.64 mm, vias 2 -> 0
- net GND_CPU: track 0.00 -> 6.19 mm, vias 0 -> 8
- net /ENC B: track 13.8 -> 7.85 mm
- net /MISO_2: track 48.5 -> 53.9 mm
- net /DRIVER IN3: track 18.8 -> 13.5 mm, vias 0 -> 1
- net /MOSI_2: track 42.4 -> 46.2 mm
- net /~{SD_CS_2}: track 43.5 -> 46.6 mm
- net Vdd: track 117.8 -> 120.3 mm, vias 2 -> 3
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- added copper zone on B.Cu, net CPU_GND_2
- added copper zone on B.Cu, net GND_CPU
- removed copper zone on B.Cu, net (none)
Other:
- board size 104.4 x 97.8 mm -> 107.2 x 104 mm
