File: Projekt3FolderyPo4Pliki/sd_i_fram/sd_i_fram.kicad_sch (KiCad schematic)
At the start: 15 parts, among them J5 Conn_02x05_Odd_Even, J6 Molex 104031

Commit message: s
Parts:
- renumbered C9 to C1, C10 to C2, J5 to J1, J6 to J2, R3 to R1, R4 to R2, R5 to R3, R6 to R4, R7 to R5, R8 to R6
Changed lines of the file:
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@@
-		)
-	)
-	(rectangle
-		(start 146.05 41.91)
-		(end 152.4 50.8)
-		(stroke
-			(width 0)
-			(type default)
-		)
-		(fill
-			(type none)
 		)
 	)
@@
 	(wire
 		(pts
-			(xy 146.05 46.99) (xy 147.32 46.99)
-		)
-		(stroke
-			(width 0)
-			(type default)
-		)
-	)
-	(wire
-		(pts
 			(xy 52.07 115.57) (xy 59.69 115.57)
 		)
@@
 	(wire
 		(pts
-			(xy 146.05 44.45) (xy 147.32 44.45)
-		)
-		(stroke
-			(width 0)
-			(type default)
-		)
-	)
-	(wire
-		(pts
 			(xy 46.99 110.49) (xy 46.99 111.76)
 		)
@@
 	(wire
 		(pts
-			(xy 146.05 49.53) (xy 147.32 49.53)
-		)
-		(stroke
-			(width 0)
-			(type default)
-		)
-	)
-	(wire
-		(pts
 			(xy 125.73 46.99) (xy 123.19 46.99)
 		)
@@
 	)
 	(label "MISO_2"
-		(at 147.32 49.53 0)
+		(at 146.05 49.53 0)
 		(effects
 			(font
@@
 	)
 	(label "MOSI_2"
-		(at 147.32 46.99 0)
+		(at 146.05 46.99 0)
 		(effects
 			(font
@@
 		)
 	)
-	(label "SPI"
-		(at 149.86 41.91 0)
-		(effects
-			(font
-				(size 1.27 1.27)
-			)
-			(justify left bottom)
-		)
-	)
 	(label "MISO_2"
 		(at 59.69 36.83 0)
@@
 	)
 	(label "SCK_2"
-		(at 147.32 44.45 0)
+		(at 146.05 44.45 0)
 		(effects
 			(font
@@
 		(in_pos_files yes)
 		(dnp no)
-		(property "Reference" "C10"
+		(property "Reference" "C2"
 			(at 47.498 104.648 0)
 			(show_name no)
@@
 		(in_pos_files yes)
 		(dnp no)
-		(property "Reference" "R3"
+		(property "Reference" "R1"
 			(at 113.538 46.99 90)
 			(show_name no)
@@
 		(in_pos_files yes)
 		(dnp no)
-		(property "Reference" "C9"
+		(property "Reference" "C1"
 			(at 145.796 32.512 90)
 			(show_name no)
@@
 		(in_pos_files yes)
 		(dnp no)
-		(property "Reference" "#PWR037"
+		(property "Reference" "#PWR07"
 			(at 38.1 88.9 0)
 			(hide yes)
@@
 		(in_pos_files yes)
 		(dnp no)
-		(property "Reference" "J6"
+		(property "Reference" "J2"
 			(at 67.31 90.17 0)
 			(show_name no)
@@
 		(in_pos_files yes)
 		(dnp no)
-		(property "Reference" "R5"
+		(property "Reference" "R3"
 			(at 123.19 54.61 0)
 			(show_name no)
@@
 		(in_pos_files yes)
 		(dnp no)
-		(property "Reference" "R8"
+		(property "Reference" "R6"
 			(at 57.404 118.11 0)
 			(show_name no)
@@
 		)
 		(instances
+			(project "sd_i_fram"
+				(path "/37281f2f-a2cb-40fa-aa8d-67b98bf89d1b"
+					(reference "H8")
+					(unit 1)
+				)
+			)
 			(project "smiw_proj"
 				(path "/b984033f-847c-449b-8f32-a23b51039886"
@@
 		(in_pos_files yes)
 		(dnp no)
-		(property "Reference" "#PWR033"
+		(property "Reference" "#PWR03"
 			(at 36.83 36.83 0)
 			(hide yes)
@@
 		(dnp no)
 		(fields_autoplaced yes)
-		(property "Reference" "R6"
+		(property "Reference" "R4"
 			(at 62.23 83.8199 0)
 			(show_name no)
@@
 		(in_pos_files yes)
 		(dnp no)
-		(property "Reference" "#PWR031"
+		(property "Reference" "#PWR01"
 			(at 135.89 34.29 0)
 			(hide yes)
@@
 		(in_pos_files yes)
 		(dnp no)
-		(property "Reference" "R4"
+		(property "Reference" "R2"
 			(at 119.38 42.418 90)
 			(show_name no)
@@
 		(in_pos_files yes)
 		(dnp no)
-		(property "Reference" "#PWR034"
+		(property "Reference" "#PWR04"
 			(at 135.89 63.5 0)
 			(hide yes)
@@
 		)
 		(instances
+			(project "sd_i_fram"
+				(path "/37281f2f-a2cb-40fa-aa8d-67b98bf89d1b"
+					(reference "H7")
+					(unit 1)
+				)
+			)
 			(project "smiw_proj"
 				(path "/b984033f-847c-449b-8f32-a23b51039886"
@@
 		(in_pos_files yes)
 		(dnp no)
-		(property "Reference" "#PWR040"
+		(property "Reference" "#PWR010"
 			(at 116.84 120.65 0)
 			(hide yes)
@@
 		(in_pos_files yes)
 		(dnp no)
-		(property "Reference" "#PWR041"
+		(property "Reference" "#PWR011"
 			(at 57.15 125.73 0)
 			(hide yes)
@@
 		)
 		(instances
+			(project "sd_i_fram"
+				(path "/37281f2f-a2cb-40fa-aa8d-67b98bf89d1b"
+					(reference "H6")
+					(unit 1)
+				)
+			)
 			(project "smiw_proj"
 				(path "/b984033f-847c-449b-8f32-a23b51039886"
@@
 		(in_pos_files yes)
 		(dnp no)
-		(property "Reference" "#PWR039"
+		(property "Reference" "#PWR09"
 			(at 27.94 111.76 0)
 			(hide yes)
@@
 		(in_pos_files yes)
 		(dnp no)
-		(property "Reference" "#PWR036"
+		(property "Reference" "#PWR06"
 			(at 124.46 62.23 0)
 			(hide yes)
@@
 		(in_pos_files yes)
 		(dnp no)
-		(property "Reference" "#PWR038"
+		(property "Reference" "#PWR08"
 			(at 38.1 101.6 0)
 			(hide yes)
@@
 		(in_pos_files yes)
 		(dnp no)
-		(property "Reference" "#PWR032"
+		(property "Reference" "#PWR02"
 			(at 48.26 34.29 0)
 			(hide yes)
@@
 		(dnp no)
 		(fields_autoplaced yes)
-		(property "Reference" "R7"
+		(property "Reference" "R5"
 			(at 45.72 91.4399 0)
 			(show_name no)
@@
 		(in_pos_files yes)
 		(dnp no)
-		(property "Reference" "#PWR035"
+		(property "Reference" "#PWR05"
 			(at 59.69 82.55 0)
 			(hide yes)
@@
 		)
 		(instances
+			(project "sd_i_fram"
+				(path "/37281f2f-a2cb-40fa-aa8d-67b98bf89d1b"
+					(reference "H5")
+					(unit 1)
+				)
+			)
 			(project "smiw_proj"
 				(path "/b984033f-847c-449b-8f32-a23b51039886"
@@
 		(in_pos_files yes)
 		(dnp no)
-		(property "Reference" "J5"
+		(property "Reference" "J1"
 			(at 52.07 32.004 0)
 			(show_name no)
