File: main/main.kicad_pcb (KiCad board)
At the start: 2 copper layers, 107.8 x 71.2 mm, 54 parts, among them J1 Conn_02x06_Odd_Even, J2 Conn_02x05_Odd_Even, J3 Conn_01x02, J4 Conn_01x02, Q1 MMBT3904, SW1 SW_Push, U1 LM2596S-5, U2 M5 Stamp-S3, U3 LD1117S33TR_SOT223, U4 LM317_SOT-223, U5 LM317_SOT-223, U6 MT3608, U7 INA219AxD, U8 MAX40200AUK

Commit message: resized. Kanapka
Parts:
- J2: moved to B.Cu
Routing:
- net GND_CPU: track 52.7 -> 41.7 mm, vias 5 -> 4
- net Vdd: track 176.9 -> 187.1 mm, vias 5 -> 6
- net /~{FRAM CS}: track 34.6 -> 44.8 mm, vias 4 -> 3
- net /MOSI: track 49.5 -> 39.3 mm, vias 4 -> 3
- net /~{SD CS}: track 43.6 -> 48.8 mm, vias 5 -> 6
- net /MISO: track 47.4 -> 42.4 mm, vias 2 -> 1
- net /SCK: vias 2 -> 1
