File: main/main.kicad_pcb (KiCad board)
At the start: 2 copper layers, 107.8 x 71.2 mm, 54 parts, among them J1 Conn_02x06_Odd_Even, J2 Conn_02x05_Odd_Even, J3 Conn_01x02, J4 Conn_01x02, Q1 MMBT3904, SW1 SW_Push, U1 LM2596S-5, U2 M5 Stamp-S3, U3 LD1117S33TR_SOT223, U4 LM317_SOT-223, U5 LM317_SOT-223, U6 MT3608, U7 INA219AxD, U8 MAX40200AUK

Commit message: zatwierdzone sprawko
Parts:
- moved R13 7.29 mm to (43.6, 43.7)
- moved D8 4.92 mm to (49.9, 43.5)
Routing:
- net 12V: track 122.8 -> 115.0 mm
- net /~{PFI}: track 28.1 -> 32.1 mm
- net /~{SD CS}: track 48.8 -> 47.8 mm, vias 6 -> 4
- net /MOSI: track 39.3 -> 39.1 mm, vias 3 -> 5
