File: motor_i_enkoder/motor_i_enkoder.kicad_pcb (KiCad board)
At the start: 2 copper layers, 61 x 40.6 mm, 17 parts, among them J1 Conn_02x06_Odd_Even, J2 Conn_02x01, SW1 EC11E15204A3, U1 L298N

Commit message: resized. Kanapka
Parts:
- J1: moved to B.Cu
- moved D1 81.8 mm to (127.3, 84.2), turned to 180 degrees
- moved D2 76.1 mm to (127.3, 79.7), turned to 180 degrees
- moved SW1 75.0 mm to (121.6, 81.6), turned to 180 degrees
- moved R1 73.7 mm to (102.6, 84.8), turned to 180 degrees
- moved D3 70.6 mm to (127.3, 75.1), turned to 180 degrees
- moved R2 69.0 mm to (102.6, 81.5), turned to 180 degrees
- moved D4 65.2 mm to (127.3, 70.6), turned to 180 degrees
- moved C2 64.6 mm to (103.1, 78.4), turned to 180 degrees
- moved J1 59.0 mm to (126.5, 66.1), turned to 0 degrees
- moved H12 55.5 mm to (137.8, 93.9)
- moved L1 50.2 mm to (116.3, 64.7), turned to 180 degrees
- moved C1 49.6 mm to (104.3, 67.7), turned to 180 degrees
- moved H10 46.0 mm to (137.4, 33.0)
- moved J2 40.7 mm to (104.4, 61.3), turned to 180 degrees
- moved U1 35.5 mm to (121.3, 47.3), turned to 180 degrees
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Routing:
- net GND_2: track 0.00 -> 12.8 mm, vias 0 -> 2
- net /ENC_B_1: track 52.6 -> 60.0 mm, vias 0 -> 4
- net /DRIVER_IN3_1: track 19.8 -> 27.0 mm, vias 1 -> 2
- net /DRIVER_IN2_1: track 30.0 -> 33.5 mm, vias 2 -> 1
- net /PWM_A_1: track 20.5 -> 23.4 mm
- net 12V_2: track 9.88 -> 7.17 mm
- net /DRIVER_IN1_1: track 23.3 -> 25.7 mm
- net /DRIVER_IN4_1: track 22.0 -> 24.4 mm
- net Net-(D2-A): track 92.3 -> 93.7 mm
- net /ENC_A_1: track 92.6 -> 93.9 mm
- net Vdd_2: track 71.5 -> 70.3 mm
- net CPU_GND_2: track 0.00 -> 0.82 mm
- net Net-(D1-A): track 54.1 -> 54.7 mm, vias 2 -> 1
Other:
- board size 61 x 40.6 mm -> 107.8 x 71.2 mm
