File: motor_i_enkoder/motor_i_enkoder.kicad_pcb (KiCad board)
At the start: 2 copper layers, 107.8 x 71.2 mm, 17 parts, among them J1 Conn_02x06_Odd_Even, J2 Conn_02x01, SW1 EC11E15204A3, U1 L298N

Commit message: zatwierdzone sprawko
Parts:
- moved J2 36.4 mm to (140.8, 58.8), turned to -90 degrees
Routing:
- net Net-(D2-A): track 93.7 -> 76.6 mm
- net Net-(D1-A): track 54.7 -> 60.9 mm, vias 1 -> 2
Changed lines of the file:
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@@
 	(footprint "Connector_PinSocket_2.54mm:PinSocket_2x01_P2.54mm_Vertical"
 		(layer "F.Cu")
-		(at 104.445 61.28995 180)
+		(at 140.8 58.84 -90)
 		(descr "Through hole straight socket strip, 2x01, 2.54mm pitch, double rows (from Kicad 4.0.7), script generated")
 		(tags "Through hole socket strip THT 2x01 2.54mm double row")
 		(property "Reference" "J2"
-			(at 3.205 1.26 0)
+			(at 3.205 1.26 90)
 			(layer "F.SilkS")
 			(effects
@@
 		)
 		(property "Value" "Conn_02x01"
-			(at -1.27 2.77 0)
+			(at -1.27 2.77 90)
 			(layer "F.Fab")
 			(effects
@@
 		)
 		(property "Datasheet" ""
-			(at 0 0 0)
+			(at 0 0 90)
 			(layer "F.Fab")
 			(hide yes)
@@
 		)
 		(property "Description" "Generic connector, double row, 02x01, this symbol is compatible with counter-clockwise, top-bottom and odd-even numbering schemes., script generated (kicad-library-utils/schlib/autogen/connector/)"
-			(at 0 0 0)
+			(at 0 0 90)
 			(layer "F.Fab")
 			(hide yes)
@@
 		)
 		(property "KiLib_Generator" "connector/pin_header_socket"
-			(at 0 0 0)
+			(at 0 0 90)
 			(layer "F.SilkS")
 			(hide yes)
@@
 		(duplicate_pad_numbers_are_jumpers no)
 		(fp_line
+			(start -3.87 1.33)
+			(end 1.33 1.33)
+			(stroke
+				(width 0.12)
+				(type solid)
+			)
+			(layer "F.SilkS")
+		)
+		(fp_line
+			(start -1.27 1.27)
+			(end 1.33 1.27)
+			(stroke
+				(width 0.12)
+				(type solid)
+			)
+			(layer "F.SilkS")
+		)
+		(fp_line
 			(start 1.33 1.27)
 			(end 1.33 1.33)
@@
 		)
 		(fp_line
+			(start -3.87 -1.33)
+			(end -3.87 1.33)
+			(stroke
+				(width 0.12)
+				(type solid)
+			)
+			(layer "F.SilkS")
+		)
+		(fp_line
+			(start -3.87 -1.33)
+			(end -1.27 -1.33)
+			(stroke
+				(width 0.12)
+				(type solid)
+			)
+			(layer "F.SilkS")
+		)
+		(fp_line
+			(start -1.27 -1.33)
+			(end -1.27 1.27)
+			(stroke
+				(width 0.12)
+				(type solid)
+			)
+			(layer "F.SilkS")
+		)
+		(fp_line
+			(start 0 -1.33)
+			(end 1.33 -1.33)
+			(stroke
+				(width 0.12)
+				(type solid)
+			)
+			(layer "F.SilkS")
+		)
+		(fp_line
 			(start 1.33 -1.33)
 			(end 1.33 0)
@@
 		)
 		(fp_line
-			(start 0 -1.33)
-			(end 1.33 -1.33)
-			(stroke
-				(width 0.12)
-				(type solid)
-			)
-			(layer "F.SilkS")
-		)
-		(fp_line
-			(start -1.27 1.27)
-			(end 1.33 1.27)
-			(stroke
-				(width 0.12)
-				(type solid)
-			)
-			(layer "F.SilkS")
-		)
-		(fp_line
-			(start -1.27 -1.33)
-			(end -1.27 1.27)
-			(stroke
-				(width 0.12)
-				(type solid)
-			)
-			(layer "F.SilkS")
-		)
-		(fp_line
-			(start -3.87 1.33)
-			(end 1.33 1.33)
-			(stroke
-				(width 0.12)
-				(type solid)
-			)
-			(layer "F.SilkS")
-		)
-		(fp_line
-			(start -3.87 -1.33)
-			(end -1.27 -1.33)
-			(stroke
-				(width 0.12)
-				(type solid)
-			)
-			(layer "F.SilkS")
-		)
-		(fp_line
-			(start -3.87 -1.33)
-			(end -3.87 1.33)
-			(stroke
-				(width 0.12)
-				(type solid)
-			)
-			(layer "F.SilkS")
+			(start -4.31 1.77)
+			(end -4.31 -1.77)
+			(stroke
+				(width 0.05)
+				(type solid)
+			)
+			(layer "F.CrtYd")
 		)
 		(fp_line
@@
 		)
 		(fp_line
+			(start -4.31 -1.77)
+			(end 1.77 -1.77)
+			(stroke
+				(width 0.05)
+				(type solid)
+			)
+			(layer "F.CrtYd")
+		)
+		(fp_line
 			(start 1.77 -1.77)
 			(end 1.77 1.77)
@@
 		)
 		(fp_line
-			(start -4.31 1.77)
-			(end -4.31 -1.77)
-			(stroke
-				(width 0.05)
-				(type solid)
-			)
-			(layer "F.CrtYd")
-		)
-		(fp_line
-			(start -4.31 -1.77)
-			(end 1.77 -1.77)
-			(stroke
-				(width 0.05)
-				(type solid)
-			)
-			(layer "F.CrtYd")
+			(start -3.81 1.27)
+			(end -3.81 -1.27)
+			(stroke
+				(width 0.1)
+				(type solid)
+			)
+			(layer "F.Fab")
 		)
 		(fp_line
@@
 		)
 		(fp_line
+			(start -3.81 -1.27)
+			(end 0.635 -1.27)
+			(stroke
+				(width 0.1)
+				(type solid)
+			)
+			(layer "F.Fab")
+		)
+		(fp_line
 			(start 0.635 -1.27)
 			(end 1.27 -0.635)
@@
 			(layer "F.Fab")
 		)
-		(fp_line
-			(start -3.81 1.27)
-			(end -3.81 -1.27)
-			(stroke
-				(width 0.1)
-				(type solid)
-			)
-			(layer "F.Fab")
-		)
-		(fp_line
-			(start -3.81 -1.27)
-			(end 0.635 -1.27)
-			(stroke
-				(width 0.1)
-				(type solid)
-			)
-			(layer "F.Fab")
-		)
 		(fp_text user "${REFERENCE}"
-			(at -1.27 0 0)
+			(at -1.27 0 90)
 			(layer "F.Fab")
 			(effects
@@
 		)
 		(pad "1" thru_hole rect
-			(at 0 0 180)
+			(at 0 0 270)
 			(size 1.7 1.7)
 			(drill 1)
@@
 		)
 		(pad "2" thru_hole circle
-			(at -2.54 0 180)
+			(at -2.54 0 270)
 			(size 1.7 1.7)
 			(drill 1)
@@
 	)
 	(gr_rect
-		(start 128.95 27.85)
-		(end 143.35 66.35)
-		(stroke
-			(width 0.2)
-			(type default)
-		)
-		(fill no)
-		(layer "Dwgs.User")
-	)
-	(gr_rect
 		(start 35.6 27.85)
 		(end 143.45 99.05)
@@
 	)
 	(segment
+		(start 133.71 58.84)
+		(end 131.72 56.85)
+		(width 0.4)
+		(layer "B.Cu")
+		(net "Net-(D2-A)")
+	)
+	(segment
+		(start 131.72 65.10995)
+		(end 131.72 56.85)
+		(width 0.4)
+		(layer "B.Cu")
+		(net "Net-(D2-A)")
+	)
+	(segment
+		(start 140.8 58.84)
+		(end 133.71 58.84)
+		(width 0.4)
+		(layer "B.Cu")
+		(net "Net-(D2-A)")
+	)
+	(segment
 		(start 121.345 49.86995)
 		(end 118.805 47.32995)
@@
 	)
 	(segment
-		(start 106.776522 48.62995)
-		(end 117.505 48.62995)
-		(width 0.4)
-		(layer "B.Cu")
-		(net "Net-(D2-A)")
-	)
-	(segment
-		(start 104.445 61.28995)
-		(end 103.535 60.37995)
-		(width 0.4)
-		(layer "B.Cu")
-		(net "Net-(D2-A)")
-	)
-	(segment
-		(start 103.535 60.37995)
-		(end 103.535 51.871472)
-		(width 0.4)
-		(layer "B.Cu")
-		(net "Net-(D2-A)")
-	)
-	(segment
 		(start 131.705 51.705)
 		(end 129.86995 49.86995)
@@
 	)
 	(segment
-		(start 103.535 51.871472)
-		(end 106.776522 48.62995)
-		(width 0.4)
-		(layer "B.Cu")
-		(net "Net-(D2-A)")
-	)
-	(segment
-		(start 131.72 65.10995)
+		(start 131.72 56.85)
 		(end 131.72 54.117183)
 		(width 0.4)
@@
 		(start 131.72 54.117183)
 		(end 131.705 54.102183)
-		(width 0.4)
-		(layer "B.Cu")
-		(net "Net-(D2-A)")
-	)
-	(segment
-		(start 117.505 48.62995)
-		(end 118.805 47.32995)
 		(width 0.4)
 		(layer "B.Cu")
@@
 	)
 	(segment
-		(start 110.785 57.48995)
-		(end 111.4 57.48995)
-		(width 0.4)
+		(start 129.65 72.85)
+		(end 129.35 73.15)
+		(width 0.6)
 		(layer "F.Cu")
 		(net "Net-(D1-A)")
@@
 	)
 	(segment
-		(start 114.995 57.48995)
-		(end 111.4 57.48995)
-		(width 0.4)
-		(layer "F.Cu")
-		(net "Net-(D1-A)")
-	)
-	(segment
-		(start 107.6 61.28995)
-		(end 106.985 61.28995)
-		(width 0.4)
-		(layer "F.Cu")
-		(net "Net-(D1-A)")
-	)
-	(segment
 		(start 124.1 66.55)
 		(end 124.1 62.56995)
@@
 	)
 	(segment
+		(start 129.35 73.15)
+		(end 129.35 75.10995)
+		(width 0.6)
+		(layer "F.Cu")
+		(net "Net-(D1-A)")
+	)
+	(segment
 		(start 127 72.75995)
 		(end 127 69.45)
@@
 	)
 	(segment
-		(start 120.075 52.40995)
-		(end 114.995 57.48995)
-		(width 0.4)
+		(start 134.1 63)
+		(end 140.8 56.3)
+		(width 0.6)
 		(layer "F.Cu")
 		(net "Net-(D1-A)")
@@
 	)
 	(via
-		(at 110.785 57.48995)
+		(at 129.65 72.85)
 		(size 0.6)
 		(drill 0.3)
@@
 		(net "Net-(D1-A)")
 	)
-	(segment
-		(start 106.985 61.28995)
-		(end 110.785 57.48995)
-		(width 0.4)
-		(layer "B.Cu")
+	(via
+		(at 134.1 63)
+		(size 0.9)
+		(drill 0.6)
+		(layers "F.Cu" "B.Cu")
 		(net "Net-(D1-A)")
+	)
+	(segment
+		(start 133.25 69.25)
+		(end 129.65 72.85)
+		(width 0.6)
+		(layer "B.Cu")
+		(net "Net-(D1-A)")
+	)
+	(segment
+		(start 133.25 63.85)
+		(end 133.25 69.25)
+		(width 0.6)
+		(layer "B.Cu")
+		(net "Net-(D1-A)")
+	)
+	(segment
+		(start 134.1 63)
+		(end 133.25 63.85)
+		(width 0.6)
+		(layer "B.Cu")
+		(net "Net-(D1-A)")
